File: electronics/expansion_card/Expansion_Card.kicad_pcb (KiCad board)
At the start: 2 copper layers, 26 x 30 mm, 11 parts, among them P1 USB_C_Plug_USB2.0, U1 AP2112K-3.3

Commit message: Updated KiCad files to match KiCad 9
Other:
- net class Default removed
